File: Hardware/Hardware.kicad_pcb (KiCad board)
At the start: 2 copper layers, 45 parts, among them J1 Conn_02x02_Odd_Even, J2 Conn_01x04, J3 Conn_02x02_Odd_Even, Q1 BD140, Q10 BC548, Q11 BD139, Q12 BD139, Q2 BD140, Q3 BC548, Q4 BC548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

Commit message: update
Parts:
- removed C1, C2: 47uF, Capacitor_SMD:CP_Elec_4x5.7
- removed HC-1: Conn_01x06_Female, Connector_PinHeader_2.54mm:PinHeader_1x06_P2.54mm_Vertical
- removed U1: LD1117S50TR_SOT223, Package_TO_SOT_SMD:SOT-223-3_TabPin2
- added J10: Conn_01x04, Connector_PinHeader_2.54mm:PinHeader_1x04_P2.54mm_Vertical, F.Cu at (165.3, 73.4)
- added J11: Conn_01x04, Connector_PinHeader_2.54mm:PinHeader_1x04_P2.54mm_Vertical, F.Cu at (152.7, 73.3)
- added J4: Conn_01x01, Connector_PinHeader_2.54mm:PinHeader_1x01_P2.54mm_Vertical, F.Cu at (87.2, 89.2)
- added J5: Conn_01x01, Connector_PinHeader_2.54mm:PinHeader_1x01_P2.54mm_Vertical, F.Cu at (131.2, 89.3)
- added J6: Conn_01x01, Connector_PinHeader_2.54mm:PinHeader_1x01_P2.54mm_Vertical, F.Cu at (87.2, 110.1)
- added J7: Conn_01x01, Connector_PinHeader_2.54mm:PinHeader_1x01_P2.54mm_Vertical, F.Cu at (131.2, 110.1)
- added J8: Conn_01x03, Connector_PinHeader_2.54mm:PinHeader_1x03_P2.54mm_Vertical, F.Cu at (194.2, 98.0)
- added J9: Conn_01x03, Connector_PinHeader_2.54mm:PinHeader_1x03_P2.54mm_Vertical, F.Cu at (190.5, 98.0)
- added U4: HC-05, Connector_PinHeader_2.54mm:PinHeader_1x06_P2.54mm_Horizontal, F.Cu at (199.3, 92.5)
- D1, D2, D3, D4: footprint Diode_SMD:D_0805_2012Metric -> Diode_THT:D_A-405_P2.54mm_Vertical_AnodeUp; moved to F.Cu
- D5, D6, D7, D8: footprint Diode_SMD:D_0805_2012Metric -> Diode_THT:D_A-405_P2.54mm_Vertical_AnodeUp
- R10, R12, R14, R15, R16, R9: footprint Resistor_SMD:R_2010_5025Metric -> Resistor_SMD:R_0805_2012Metric; moved to B.Cu
- R11, R13: value 30k -> 15k; footprint Resistor_SMD:R_2010_5025Metric -> Resistor_SMD:R_0805_2012Metric; moved to B.Cu
- R5, R6, R7, R8: moved to B.Cu
- U3: footprint Package_DIP:DIP-14_W8.89mm_SMDSocket_LongPads -> Package_SO:SOIC-14_3.9x8.7mm_P1.27mm; moved to B.Cu
- moved R11 124.9 mm to (108.9, 106.9)
- moved R14 121.3 mm to (100.1, 96.0), turned to 90 degrees
- moved R15 119.8 mm to (100.0, 106.8), turned to 270 degrees
- moved R12 119.6 mm to (102.3, 99.8), turned to 270 degrees
- moved R9 119.0 mm to (105.3, 106.9)
- moved R16 117.7 mm to (100.1, 99.8), turned to 270 degrees
- moved R13 116.2 mm to (100.0, 103.4), turned to 90 degrees
- moved R10 106.0 mm to (105.3, 95.1)
- moved Q10 102.1 mm to (183.1, 115.1), turned to 270 degrees
- moved R8 92.8 mm to (168.8, 120.2), turned to 180 degrees
- moved U2 80.1 mm to (134.9, 100.6), turned to 90 degrees
- moved U3 78.3 mm to (108.2, 101.0), turned to 270 degrees
- moved R5 77.1 mm to (186.3, 106.9)
- moved J2 75.8 mm to (82.6, 94.8)
- moved Q12 75.0 mm to (164.0, 117.3)
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Connections:
- R1 pad 2: PWM1 -> PWM1N
- R10 pad 1: ADC0 -> ADC1
- R2 pad 1: PWM1N -> PWM1
- R5 pad 2: PWM2 -> PWM2N
- R6 pad 1: PWM2N -> PWM2
- R9 pad 1: ADC1 -> ADC0
- U2 pad 15: Net-(U2-Pad15) -> D1
- U2 pad 16: Net-(U2-Pad16) -> D0
- U2 pad 18: Net-(U2-Pad18) -> +3V3
- U2 pad 19: GND -> GNDD
- U2 pad 20: GND -> GNDD
- U2 pad 27: Net-(U2-Pad27) -> Echo0
- U2 pad 28: Net-(U2-Pad28) -> Trig0
- U2 pad 32: Net-(U2-Pad32) -> Echo1
- U2 pad 33: Net-(U2-Pad33) -> Trig1
- U3 pad 1: ADC0 -> ADC1
- U3 pad 12: (no net) -> Net-(R13-Pad1)
- U3 pad 13: (no net) -> Net-(R11-Pad1)
- U3 pad 14: (no net) -> ADC0
- U3 pad 5: Net-(R13-Pad1) -> (no net)
- U3 pad 6: Net-(R11-Pad1) -> (no net)
- U3 pad 7: ADC1 -> (no net)
Routing:
- net GND: track 38.2 -> 341.6 mm, vias 0 -> 2
- net +BATT: track 24.1 -> 255.9 mm, vias 0 -> 4
- net +5V: track 0.00 -> 165.0 mm
- net PWM1: track 0.00 -> 88.6 mm, vias 0 -> 4
- net TXB: track 0.00 -> 81.3 mm
- net PWM2: track 0.00 -> 68.3 mm
- net ADC0: track 0.00 -> 67.0 mm
- net RXB: track 0.00 -> 66.3 mm
- net ADC1: track 0.00 -> 59.6 mm
- net PWM2N: track 0.00 -> 31.8 mm
- net Net-(Q11-Pad3): track 0.00 -> 29.9 mm, vias 0 -> 2
- net D1: track 0.00 -> 25.6 mm
- net Net-(Q12-Pad3): track 0.00 -> 21.2 mm, vias 0 -> 2
- net BATMed: track 0.00 -> 21.0 mm, vias 0 -> 2
- net Net-(D6-Pad1): track 0.00 -> 20.1 mm
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- added copper zone on B.Cu, net GND
Other:
- board outline added: 125.3 x 55.9 mm
- net class Default: clearance 0.3048 -> 0.1048
- rule trace_clearance: 0.3048 -> 0.1048
- board text added: "D0 GND +3,3"
- board text added: "GND EC TG 5V"
- board text added: "IN+"
- board text added: "IN-"
