File: Hardware/Hardware.sch (KiCad schematic (older format))
At the start: 45 parts, among them J1 Conn_02x02_Odd_Even, J2 Conn_01x04, J3 Conn_02x02_Odd_Even, Q1 BD140, Q10 BC548, Q11 BD139, Q12 BD139, Q2 BD140, Q3 BC548, Q4 BC548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

Commit message: update
Parts:
- removed C1, C2: 47uF, Capacitor_SMD:CP_Elec_4x5.7, symbol Device:CP
- removed HC-1: Conn_01x06_Female, Connector_PinHeader_2.54mm:PinHeader_1x06_P2.54mm_Vertical, symbol Connector:Conn_01x06_Female
- removed U1: LD1117S50TR_SOT223, Package_TO_SOT_SMD:SOT-223-3_TabPin2, symbol Regulator_Linear:LD1117S50TR_SOT223
- added J10, J11: Conn_01x04, Connector_PinHeader_2.54mm:PinHeader_1x04_P2.54mm_Vertical, symbol Connector_Generic:Conn_01x04
- added J4, J5, J6, J7: Conn_01x01, Connector_PinHeader_2.54mm:PinHeader_1x01_P2.54mm_Vertical, symbol Connector_Generic:Conn_01x01
- added J8, J9: Conn_01x03, Connector_PinHeader_2.54mm:PinHeader_1x03_P2.54mm_Vertical, symbol Connector_Generic:Conn_01x03
- added U4: HC-05, Connector_PinHeader_2.54mm:PinHeader_1x06_P2.54mm_Horizontal, symbol HC-05:HC-05
- D1, D2, D3, D4, D5, D6, D7, D8: footprint Diode_SMD:D_0805_2012Metric -> Diode_THT:D_A-405_P2.54mm_Vertical_AnodeUp
- R10, R12, R14, R15, R16, R9: footprint Resistor_SMD:R_2010_5025Metric -> Resistor_SMD:R_0805_2012Metric
- R11, R13: value 30k -> 15k; footprint Resistor_SMD:R_2010_5025Metric -> Resistor_SMD:R_0805_2012Metric
- U3: footprint Package_DIP:DIP-14_W8.89mm_SMDSocket_LongPads -> Package_SO:SOIC-14_3.9x8.7mm_P1.27mm
Connections:
- net +5V: now also J10.1 (Pin_1), J11.1 (Pin_1), J5.1 (Pin_1), U4.5 (Pin_5)
- net +BATT: now also J4.1 (Pin_1)
- net ADC0: now also R9.1, U3.14; no longer R10.1, U3.1
- net ADC1: now also R10.1, U3.1; no longer R9.1, U3.7
- net GND: now also J10.4 (Pin_4), J11.4 (Pin_4), J6.1 (Pin_1), J7.1 (Pin_1), U4.4 (Pin_4); no longer U2.19 (GND), U2.20 (GND)
- net PWM1: now also R2.1; no longer R1.2
- net PWM1N: now also R1.2; no longer R2.1
- net PWM2: now also R6.1; no longer R5.2
- net PWM2N: now also R5.2; no longer R6.1
- net RXB: now also U4.2 (Pin_2)
- net TXB: now also U4.3 (Pin_3)
- net D1: now reaches U2.15 (PB10_SCL2)
- net D1: now also J8.3 (Pin_3)
- net D0: now reaches U2.16 (PB11_SDA2)
- net D0: now also J9.3 (Pin_3)
- net +3V3: now reaches U2.18 (VCC3V3)
- net +3V3: now also J8.1 (Pin_1), J9.1 (Pin_1)
- net Echo0: now reaches U2.27 (PA10_RX1)
- net Echo0: now also J10.3 (Pin_3)
- net Trig0: now reaches U2.28 (PA11_USB_D-)
- net Trig0: now also J10.2 (Pin_2)
- net Echo1: now reaches U2.32 (PB4)
- net Echo1: now also J11.3 (Pin_3)
- net Trig1: now reaches U2.33 (PB5)
- net Trig1: now also J11.2 (Pin_2)
- net at R11.1, R9.2: now also U3.13 (-); no longer U3.6 (-)
- net at R13.1, R15.1: now also U3.12 (+); no longer U3.5 (+)
- new net GNDD: J8.2 (Pin_2), J9.2 (Pin_2), U2.19 (GND), U2.20 (GND)
Other:
- note added: "Encoder velocidade"
